File: LedDriver/LedDriver.kicad_sch (KiCad schematic)
At the start: 23 parts, among them J2 Micro_SD_Card_Det1, Y1 32.768 kHz

Commit message: Update to Add Known JST3 Pin thingys
Parts:
- added J3: (no value), symbol JSTCons:5Pin
Connections:
- net USBDM: now also J1.1; no longer J1.5
- net USBDP: now also J1.2; no longer J1.4
- net JST3PIN4: now reaches R12.1
- net JST3PIN4: now also J3.4
Other:
- moved on the sheet: J1
Changed lines of the file:
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@@
-	(wire
-		(pts
-			(xy 262.89 30.48) (xy 271.78 30.48)
-		)
-		(stroke
-			(width 0)
-			(type default)
-		)
-	)
 	(wire
 		(pts
@@
 	(wire
 		(pts
+			(xy 262.89 30.48) (xy 273.05 30.48)
+		)
+		(stroke
+			(width 0)
+			(type default)
+		)
+	)
+	(wire
+		(pts
 			(xy 218.44 144.78) (xy 214.63 144.78)
 		)
@@
 	(wire
 		(pts
-			(xy 262.89 33.02) (xy 271.78 33.02)
-		)
-		(stroke
-			(width 0)
-			(type default)
-		)
-	)
-	(wire
-		(pts
 			(xy 45.72 73.66) (xy 58.42 73.66)
 		)
@@
 		(pts
 			(xy 45.72 91.44) (xy 58.42 91.44)
+		)
+		(stroke
+			(width 0)
+			(type default)
+		)
+	)
+	(wire
+		(pts
+			(xy 262.89 33.02) (xy 273.05 33.02)
 		)
 		(stroke
@@
 		)
 	)
+	(global_label "JST3PIN4"
+		(shape input)
+		(at 273.05 54.61 180)
+		(fields_autoplaced yes)
+		(effects
+			(font
+				(size 1.27 1.27)
+			)
+			(justify right)
+		)
+		(property "Intersheetrefs" "${INTERSHEET_REFS}"
+			(at 261.2958 54.61 0)
+			(hide yes)
+			(show_name no)
+			(do_not_autoplace no)
+			(effects
+				(font
+					(size 1.27 1.27)
+				)
+				(justify right)
+			)
+		)
+	)
 	(global_label "USBDM"
 		(shape input)
@@
 	(global_label "USBDP"
 		(shape input)
-		(at 262.89 30.48 180)
+		(at 262.89 33.02 180)
 		(fields_autoplaced yes)
 		(effects
@@
 		)
 		(property "Intersheetrefs" "${INTERSHEET_REFS}"
-			(at 253.5548 30.48 0)
+			(at 253.5548 33.02 0)
 			(hide yes)
 			(show_name no)
@@
 	(global_label "USBDM"
 		(shape input)
-		(at 262.89 33.02 180)
+		(at 262.89 30.48 180)
 		(fields_autoplaced yes)
 		(effects
@@
 		)
 		(property "Intersheetrefs" "${INTERSHEET_REFS}"
-			(at 253.3734 33.02 0)
+			(at 253.3734 30.48 0)
+			(hide yes)
+			(show_name no)
+			(do_not_autoplace no)
+			(effects
+				(font
+					(size 1.27 1.27)
+				)
+				(justify right)
+			)
+		)
+	)
+	(global_label "JST3PIN4"
+		(shape input)
+		(at 77.47 123.19 270)
+		(fields_autoplaced yes)
+		(effects
+			(font
+				(size 1.27 1.27)
+			)
+			(justify right)
+		)
+		(property "Intersheetrefs" "${INTERSHEET_REFS}"
+			(at 77.47 134.9442 90)
 			(hide yes)
 			(show_name no)
@@
 	(symbol
 		(lib_id "JSTCons:5Pin")
-		(at 274.32 33.02 0)
+		(at 275.59 40.64 0)
 		(unit 1)
 		(body_style 1)
@@
 		(fields_autoplaced yes)
 		(property "Reference" "J1"
-			(at 279.4 27.9399 0)
+			(at 280.67 35.5599 0)
 			(show_name no)
 			(do_not_autoplace no)
@@
 		)
 		(property "Value" ""
-			(at 274.32 33.02 0)
+			(at 275.59 40.64 0)
 			(show_name no)
 			(do_not_autoplace no)
@@
 		)
 		(property "Footprint" ""
-			(at 274.32 33.02 0)
+			(at 275.59 40.64 0)
 			(hide yes)
 			(show_name no)
@@
 		)
 		(property "Datasheet" ""
-			(at 274.32 33.02 0)
+			(at 275.59 40.64 0)
 			(hide yes)
 			(show_name no)
@@
 		)
 		(property "Description" ""
-			(at 274.32 33.02 0)
+			(at 275.59 40.64 0)
 			(hide yes)
 			(show_name no)
@@
 					(unit 1)
 				)
+			)
+		)
+	)
+	(symbol
+		(lib_id "JSTCons:5Pin")
+		(at 275.59 57.15 0)
+		(unit 1)
+		(body_style 1)
+		(exclude_from_sim no)
+		(in_bom yes)
+		(on_board yes)
+		(in_pos_files yes)
+		(dnp no)
+		(fields_autoplaced yes)
+		(property "Reference" "J3"
+			(at 280.67 52.0699 0)
+			(show_name no)
+			(do_not_autoplace no)
+			(effects
+				(font
+					(size 1.27 1.27)
+				)
+				(justify left)
+			)
+		)
+		(property "Value" ""
+			(at 275.59 57.15 0)
+			(show_name no)
+			(do_not_autoplace no)
+			(effects
+				(font
+					(size 1.27 1.27)
+				)
+			)
+		)
+		(property "Footprint" ""
+			(at 275.59 57.15 0)
+			(hide yes)
+			(show_name no)
+			(do_not_autoplace no)
+			(effects
+				(font
+					(size 1.27 1.27)
+				)
+			)
+		)
+		(property "Datasheet" ""
+			(at 275.59 57.15 0)
+			(hide yes)
+			(show_name no)
+			(do_not_autoplace no)
+			(effects
+				(font
+					(size 1.27 1.27)
+				)
+			)
+		)
+		(property "Description" ""
+			(at 275.59 57.15 0)
+			(hide yes)
+			(show_name no)
+			(do_not_autoplace no)
+			(effects
+				(font
+					(size 1.27 1.27)
+				)
+			)
+		)
+		(pin "5"
+		)
+		(pin "2"
+		)
+		(pin "1"
+		)
+		(pin "3"
+		)
+		(pin "4"
+		)
+		(instances
+			(project "LedDriver"
+				(path "/b8b1ee11-cbc7-4ed7-a3ef-d663a64fa814"
+					(reference "J3")
+					(unit 1)
+				)
